Commit message: updated for fardin vai

File: install/test_bot/share/test_bot/description/robot_core.xacro (robot description, xacro)
@@ -41,7 +41,4 @@
         </xacro:inertial_box>
     </link>
-    <gazebo reference="chassis">
-        <material>Gazebo/White</material>
-    </gazebo>
     <!-- LEFT WHEEL LINK -->
     <joint name="left_wheel_joint" type="continuous">
