Commit message: corrected inertia tags

File: description/robot_core.xacro (robot description, xacro)
@@ -2,14 +2,14 @@
 <robot xmlns:xacro="http://www.ros.org/wiki/xacro" >
     <xacro:include filename="inertial_macros.xacro"/>
-    <material name = "white">
-        <color rgba="1 1 1 1"/>
+    <material name="white">
+        <color rgba="1 1 1 1" />
     </material>
-    <material name = "orange">
+    <material name="orange">
         <color rgba="1 0.3 0.1 1"/>
     </material>
-    <material name = "blue">
+    <material name="blue">
         <color rgba="0.2 0.2 1 1"/>
     </material>
-    <material name = "black">
+    <material name="black">
         <color rgba="0 0 0 1"/>
     </material>
@@ -17,13 +17,13 @@
     <link name="base_link">
     </link>
-    <!-- CHASSIS LINK   -->
+    <!-- CHASSIS LINK -->
     <joint name="chassis_joint" type="fixed">
         <parent link="base_link"/>
         <child link="chassis"/>
-        <origin xyz="-0.1 0.0 0.0"/>
+        <origin xyz="-0.1 0 0"/>
     </joint>
     <link name="chassis">
         <visual>
-            <origin xyz="0.15 0.0 0.075"/>
+            <origin xyz="0.15 0 0.075"/>
             <geometry>
                 <box size="0.3 0.3 0.15"/>
@@ -32,19 +32,19 @@
         </visual>
         <collision>
-            <origin xyz="0.15 0.0 0.075"/>
+            <origin xyz="0.15 0 0.075"/>
             <geometry>
                 <box size="0.3 0.3 0.15"/>
             </geometry>
         </collision>
-        <xacro:inertial_box mass = "0.5", x="0.3", y="0.3" z="0.15">
-            <origin xyz="0.15 0.0 0.075", rpy="0.0 0.0 0.0"/>
+        <xacro:inertial_box mass="0.5" x="0.3" y="0.3" z="0.15">
+            <origin xyz="0.15 0 0.075" rpy="0 0 0"/>
         </xacro:inertial_box>
     </link>
-    <!-- LEFT WHEEL LINK  -->
+    <!-- LEFT WHEEL LINK -->
     <joint name="left_wheel_joint" type="continuous">
         <parent link="base_link"/>
         <child link="left_wheel"/>
-        <origin xyz="0.0 0.175 0.0" rpy="-${pi/2} 0.0 0.0"/>
-        <axis xyz="0.0 0.0 1"/>
+        <origin xyz="0 0.175 0" rpy="-${pi/2} 0 0" />
+        <axis xyz="0 0 1"/>
     </joint>
     <link name="left_wheel">
@@ -60,14 +60,14 @@
             </geometry>
         </collision>
-        <xacro:inertial_cylinder mass = "0.1", length = "0.04", radius = "0.05">
-            <origin xyz="0.0 0.175 0.0" rpy="-${pi/2} 0.0 0.0"/>
+        <xacro:inertial_cylinder mass="0.1" length="0.04" radius="0.05">
+            <origin xyz="0 0 0" rpy="0 0 0"/>
         </xacro:inertial_cylinder>
     </link>
-        <!-- RIGHT WHEEL LINK  -->
+    <!-- RIGHT WHEEL LINK -->
     <joint name="right_wheel_joint" type="continuous">
         <parent link="base_link"/>
         <child link="right_wheel"/>
-        <origin xyz="0.0 -0.175 0.0" rpy="${pi/2} 0.0 0.0"/>
-        <axis xyz="0.0 0.0 -1"/>
+        <origin xyz="0 -0.175 0" rpy="${pi/2} 0 0" />
+        <axis xyz="0 0 -1"/>
     </joint>
     <link name="right_wheel">
@@ -83,13 +83,13 @@
             </geometry>
         </collision>
-        <xacro:inertial_cylinder mass = "0.1", length = "0.04", radius = "0.05">
-            <origin xyz="0.0 -0.175 0.0" rpy="${pi/2} 0.0 0.0"/>
+        <xacro:inertial_cylinder mass="0.1" length="0.04" radius="0.05">
+            <origin xyz="0 0 0" rpy="0 0 0"/>
         </xacro:inertial_cylinder>
     </link>
-    <!-- CASTER WHEEL LINK  -->
-    <joint name="caster_wheel" type="fixed">
+    <!-- CASTER WHEEL LINK -->
+    <joint name="caster_wheel_joint" type="fixed">
         <parent link="chassis"/>
         <child link="caster_wheel"/>
-        <origin xyz="0.24 0.0 0.0"/>
+        <origin xyz="0.24 0 0"/>
     </joint>
     <link name="caster_wheel">
@@ -105,6 +105,6 @@
             </geometry>
         </collision>
-        <xacro:inertial_sphere mass = "0.1", radius = "0.05">
-            <origin xyz="0.24 0.0 0.0"/>
+        <xacro:inertial_sphere mass="0.1" radius="0.05">
+            <origin xyz="0 0 0" rpy="0 0 0"/>
         </xacro:inertial_sphere>
     </link>

Commit message: added gazebo control plugin and moved with keyboard in gazebo

File: description/robot_core.xacro (robot description, xacro)
@@ -67,4 +67,7 @@
         </xacro:inertial_cylinder>
     </link>
+    <gazebo reference="left_wheel">
+        <material>Gazebo/Blue</material>
+    </gazebo>
     <!-- RIGHT WHEEL LINK -->
     <joint name="right_wheel_joint" type="continuous">
@@ -90,4 +93,7 @@
         </xacro:inertial_cylinder>
     </link>
+    <gazebo reference="right_wheel">
+        <material>Gazebo/Blue</material>
+    </gazebo>
     <!-- CASTER WHEEL LINK -->
     <joint name="caster_wheel_joint" type="fixed">
@@ -112,3 +118,8 @@
         </xacro:inertial_sphere>
     </link>
+    <gazebo reference="caster_wheel">
+        <material>Gazebo/Black</material>
+        <mu1>0.001</mu1>
+        <mu2>0.001</mu2>
+    </gazebo>
 </robot>

Commit message: updated till motor testing

File: description/robot_core.xacro (robot description, xacro)
@@ -2,17 +2,17 @@
 <robot xmlns:xacro="http://www.ros.org/wiki/xacro">
     <xacro:include filename="inertial_macros.xacro"/>
-    <xacro:property name="chassis_length" value="0.335"/>
-    <xacro:property name="chassis_width" value="0.265"/>
-    <xacro:property name="chassis_height" value="0.138"/>
+    <xacro:property name="chassis_length" value="0.485"/>
+    <xacro:property name="chassis_width" value="0.240"/>
+    <xacro:property name="chassis_height" value="0.350"/>
     <xacro:property name="chassis_mass" value="1.0"/>
     <xacro:property name="wheel_radius" value="0.065"/>
-    <xacro:property name="wheel_thickness" value="0.026"/>
+    <xacro:property name="wheel_thickness" value="0.055"/>
     <xacro:property name="wheel_mass" value="0.05"/>
-    <xacro:property name="wheel_offset_x" value="0.226"/>
-    <xacro:property name="wheel_offset_y" value="0.1485"/>
-    <xacro:property name="wheel_offset_z" value="0.01"/>
-    <xacro:property name="caster_wheel_radius" value="0.01"/>
+    <xacro:property name="wheel_offset_x" value="0.045"/>
+    <xacro:property name="wheel_offset_y" value="0.1765"/>
+    <xacro:property name="wheel_offset_z" value="0.037"/>
+    <xacro:property name="caster_wheel_radius" value="0.050"/>
     <xacro:property name="caster_wheel_mass" value="0.01"/>
-    <xacro:property name="caster_wheel_offset_x" value="0.075"/>
+    <xacro:property name="caster_wheel_offset_x" value="0.420"/>
     <xacro:property name="caster_wheel_offset_z" value="${wheel_offset_z - wheel_radius + caster_wheel_radius}"/>
     <material name="white">
